File: guitar-pedal.kicad_pcb (KiCad board)
At the start: 2 copper layers, 50 parts, among them J1 USB_OTG, J2 AudioJack2, J3 AudioJack2, J4 Test_Headers, SW1 SW_SPDT, SW2 SW_3PDT, SW3 Boot, SW4 Reset, SW5 SW_Push_SPDT, SW6 SW_Push_SPDT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

Commit message: no seriously, get started on layout
Parts:
- J4: footprint Connector_PinHeader_2.54mm:PinHeader_1x10_P2.54mm_Vertical -> Connector_PinHeader_2.54mm:PinHeader_2x05_P2.54mm_Vertical
- SW3: footprint Resistor_SMD:R_0603_1608Metric_Pad0.98x0.95mm_HandSolder -> Connector_PinHeader_2.54mm:PinHeader_1x02_P2.54mm_Vertical
- moved SW6 97.9 mm to (131.4, 161.3)
- moved SW2 95.4 mm to (141.6, 164.5), turned to 90 degrees
- moved C13 87.8 mm to (90.2, 68.6)
- moved J4 87.8 mm to (200.7, 129.5)
- moved D1 86.8 mm to (149.2, 153.7)
- moved U1 86.5 mm to (201.9, 81.3)
- moved R8 84.8 mm to (87.6, 53.3)
- moved SW1 84.6 mm to (158.8, 152.4)
- moved C7 81.9 mm to (94.0, 52.1)
- moved R9 79.1 mm to (159.5, 171.4)
- moved SW5 76.3 mm to (171.4, 161.3)
- moved C8 74.2 mm to (90.2, 58.4)
- moved C14 73.7 mm to (90.2, 63.5)
- moved C3 68.6 mm to (212.1, 81.3)
- moved POT4 62.3 mm to (157.5, 141.0)
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
Commit message: wip traces and layout
Parts:
- moved J4 116.3 mm to (84.5, 125.1)
- moved C15 78.9 mm to (112.6, 127.3), turned to -90 degrees
- moved R7 77.3 mm to (155.6, 134.6)
- moved C17 76.7 mm to (110.1, 111.5), turned to 90 degrees
- moved C3 76.3 mm to (155.6, 132.6)
- moved C12 75.6 mm to (114.7, 127.0), turned to -90 degrees
- moved C21 74.6 mm to (120.4, 132.5), turned to -90 degrees
- moved C20 73.0 mm to (118.2, 131.2), turned to -90 degrees
- moved C16 72.9 mm to (112.9, 111.5), turned to 90 degrees
- moved C18 72.4 mm to (116.5, 127.0), turned to -90 degrees
- moved C1 71.0 mm to (142.6, 136.3)
- moved U1 69.6 mm to (151.8, 129.5)
- moved C19 69.2 mm to (115.4, 111.5), turned to 90 degrees
- moved U4 68.6 mm to (117.7, 119.6), turned to 90 degrees
- moved R1 67.5 mm to (142.6, 127.2), turned to 180 degrees
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Routing:
- net +3V3: track 0.00 -> 61.9 mm
- net Net-(C8-Pad1): track 0.00 -> 13.3 mm, vias 0 -> 2
- net Net-(C21-Pad1): track 0.00 -> 9.77 mm
- net +5V: track 0.00 -> 8.13 mm
- net Net-(C20-Pad1): track 0.00 -> 7.88 mm
- net Net-(C5-Pad2): track 0.00 -> 6.90 mm
- net Net-(C3-Pad1): track 0.00 -> 5.27 mm
- net Net-(C19-Pad1): track 0.00 -> 4.09 mm
- net Net-(C22-Pad1): track 0.00 -> 4.06 mm
- net Net-(C18-Pad1): track 0.00 -> 3.47 mm
- net Net-(C1-Pad1): track 0.00 -> 2.31 mm
- net /SWITCHED_IN: track 0.00 -> 2.29 mm
- net /SWITCHED_OUT: track 0.00 -> 2.05 mm
- net /CODEC_A_IN: track 0.00 -> 0.65 mm

Commit message: slight layout progress
Parts:
- moved C6 17.8 mm to (126.7, 100.1), turned to 90 degrees
- moved C7 10.2 mm to (129.8, 100.1), turned to 90 degrees
- moved C13 9.82 mm to (132.6, 95.1), turned to 90 degrees
- moved R8 7.02 mm to (132.6, 100.1), turned to 90 degrees
- moved C11 6.17 mm to (158.8, 113.4), turned to -90 degrees
- moved C14 6.07 mm to (135.2, 95.1), turned to 90 degrees
- moved C8 5.88 mm to (135.1, 99.9), turned to -90 degrees
- moved C10 1.48 mm to (119.6, 91.4)
- moved J1 0.41 mm to (136.5, 66.3)
Routing:
- net +3V3: track 61.9 -> 35.9 mm
- net Net-(C8-Pad1): track 13.3 -> 6.37 mm, vias 2 -> 0
Other:
- board outline added: 63 x 117.1 mm

Commit message: layout: wired pots sort of
Parts:
- SW3: footprint Connector_PinHeader_2.54mm:PinHeader_1x02_P2.54mm_Vertical -> Resistor_SMD:R_0603_1608Metric_Pad0.98x0.95mm_HandSolder
- moved J4 33.0 mm to (112.0, 143.3)
- moved R9 9.19 mm to (145.3, 176.8), turned to 90 degrees
- moved SW6 7.53 mm to (116.8, 167.7)
- moved SW2 7.12 mm to (127.5, 172.7)
- moved SW5 6.90 mm to (157.5, 167.7)
- moved D1 6.52 mm to (135.6, 161.5), turned to 90 degrees
- moved J3 5.85 mm to (116.3, 66.5), turned to -90 degrees
- moved C11 3.57 mm to (161.4, 115.8)
- moved C8 3.57 mm to (137.8, 102.3)
- moved R8 3.57 mm to (135.3, 102.4)
- moved U3 3.57 mm to (149.9, 108.4)
- moved C13 3.57 mm to (135.3, 97.5)
- moved C14 3.57 mm to (137.8, 97.5)
- moved C6 3.57 mm to (129.4, 102.5)
- moved C7 3.57 mm to (132.5, 102.4)
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Connections:
- POT1 pad 2: Net-(POT1-Pad2) -> /POT1_P
- POT2 pad 2: Net-(POT2-Pad2) -> /POT2_P
- POT3 pad 2: Net-(POT3-Pad2) -> /POT3_P
- POT4 pad 2: Net-(POT4-Pad2) -> /POT4_P
- POT5 pad 2: Net-(POT5-Pad2) -> /POT5_P
- POT6 pad 2: Net-(POT6-Pad2) -> /POT6_P
- U3 pad 15: Net-(POT3-Pad2) -> unconnected-(U3-Pad15)
- U3 pad 34: unconnected-(U3-Pad34) -> /POT1_P
- U3 pad 35: unconnected-(U3-Pad35) -> /POT2_P
- U3 pad 36: unconnected-(U3-Pad36) -> /POT3_P
- U3 pad 37: unconnected-(U3-Pad37) -> /POT4_P
- U3 pad 38: Net-(POT2-Pad2) -> /POT5_P
- U3 pad 39: Net-(POT1-Pad2) -> /POT6_P
- U3 pad 4: Net-(POT4-Pad2) -> unconnected-(U3-Pad4)
- U3 pad 5: Net-(POT5-Pad2) -> unconnected-(U3-Pad5)
- U3 pad 6: Net-(POT6-Pad2) -> unconnected-(U3-Pad6)
Routing:
- net /POT3_P: track 0.00 -> 68.2 mm
- net /POT6_P: track 0.00 -> 54.8 mm
- net /POT2_P: track 0.00 -> 54.1 mm
- net /RAW_OUT: track 0.00 -> 53.1 mm
- net /SWITCHED_OUT: track 2.05 -> 49.7 mm
- net /POT1_P: track 0.00 -> 41.9 mm
- net /SWITCHED_IN: track 2.29 -> 43.0 mm
- net /POT5_P: track 0.00 -> 40.6 mm
- net /POT4_P: track 0.00 -> 28.5 mm
- net Net-(D1-Pad1): track 0.00 -> 21.1 mm
- net Net-(D1-Pad3): track 0.00 -> 12.0 mm
- net Net-(R9-Pad2): track 0.00 -> 3.16 mm

Commit message: layout progress!
Parts:
- SW3: footprint Resistor_SMD:R_0603_1608Metric_Pad0.98x0.95mm_HandSolder -> Connector_PinHeader_2.54mm:PinHeader_1x02_P2.54mm_Vertical
- moved C10 69.3 mm to (155.8, 150.6)
- moved C9 69.3 mm to (146.0, 150.6)
- moved U2 69.3 mm to (151.7, 151.7)
- moved U1 28.3 mm to (132.4, 150.2)
- moved C3 28.3 mm to (136.2, 153.3)
- moved R7 28.3 mm to (136.2, 155.3)
- moved C1 23.8 mm to (125.1, 152.3)
- moved C4 23.8 mm to (125.1, 154.6)
- moved C5 23.8 mm to (125.1, 147.8)
- moved R1 23.8 mm to (125.1, 143.2)
- moved R3 23.8 mm to (125.1, 150.1)
- moved R5 23.8 mm to (125.1, 145.5)
- moved R9 12.5 mm to (144.4, 164.3), turned to 180 degrees
- moved SW1 10.8 mm to (141.0, 161.3), turned to 90 degrees
- moved D1 9.89 mm to (125.7, 161.3)
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Connections:
- U3 pad 10: /CODEC_MC -> /CODEC_ZFLG
- U3 pad 11: /CODEC_SYSCLK -> /CODEC_DATA_IN
- U3 pad 17: /CODEC_RST -> /CODEC_DATA_OUT
- U3 pad 18: /CODEC_ML -> /CODEC_BITCLK
- U3 pad 20: /CODEC_BITCLK -> /CODEC_SYSCLK
- U3 pad 21: /CODEC_DATA_OUT -> /CODEC_ML
- U3 pad 22: /CODEC_DATA_IN -> /CODEC_RST
- U3 pad 8: /CODEC_ZFLG -> /CODEC_MC
Routing:
- net +3V3: track 35.9 -> 190.3 mm, vias 0 -> 2
- net /RAW_IN: track 0.00 -> 147.0 mm
- net Net-(J1-Pad1): track 0.00 -> 128.2 mm, vias 0 -> 1
- net Net-(SW5-Pad2): track 0.00 -> 74.3 mm, vias 0 -> 1
- net /RAW_OUT: track 53.1 -> 115.4 mm
- net Net-(C11-Pad2): track 0.00 -> 52.4 mm
- net /D+: track 0.00 -> 50.1 mm, vias 0 -> 2
- net /D-: track 0.00 -> 48.1 mm, vias 0 -> 2
- net +5V: track 8.13 -> 55.2 mm
- net Net-(C8-Pad1): track 6.37 -> 42.0 mm
- net /SWITCHED_OUT: track 49.7 -> 16.0 mm
- net /CODEC_RST: track 0.00 -> 29.9 mm
- net /CODEC_ML: track 0.00 -> 27.4 mm
- net /CODEC_SYSCLK: track 0.00 -> 24.9 mm
- net /CODEC_LRCLK: track 0.00 -> 22.5 mm
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Other:
- board size 63 x 117.1 mm -> 52.1 x 107.9 mm

Commit message: tiny changes
Routing:
- net /SWITCHED_OUT: track 16.0 -> 73.3 mm, vias 0 -> 2
Changed lines of the file:
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@@
   (segment (start 135.475499 153.253202) (end 136.999499 151.729202) (width 0.2032) (layer "F.Cu") (net 3))
   (segment (start 136.999499 151.358001) (end 136.171701 150.530203) (width 0.2032) (layer "F.Cu") (net 3))
+  (segment (start 137.099999 153.253202) (end 138.176 152.177201) (width 0.2032) (layer "F.Cu") (net 4))
+  (segment (start 125.222 105.156) (end 124.46 105.156) (width 0.2032) (layer "F.Cu") (net 4))
+  (segment (start 124.46 105.156) (end 123.698 105.918) (width 0.2032) (layer "F.Cu") (net 4))
   (segment (start 133.37 167.64) (end 133.37 159.065201) (width 0.2032) (layer "F.Cu") (net 4))
+  (segment (start 123.698 105.918) (end 123.698 107.495) (width 0.2032) (layer "F.Cu") (net 4))
   (segment (start 133.37 159.065201) (end 137.149999 155.285202) (width 0.2032) (layer "F.Cu") (net 4))
   (segment (start 137.149999 153.303202) (end 137.099999 153.253202) (width 0.2032) (layer "F.Cu") (net 4))
+  (segment (start 138.176 152.177201) (end 138.176 150.114) (width 0.2032) (layer "F.Cu") (net 4))
   (segment (start 137.149999 155.285202) (end 137.149999 153.303202) (width 0.2032) (layer "F.Cu") (net 4))
+  (via (at 125.222 105.156) (size 0.7112) (drill 0.3048) (layers "F.Cu" "B.Cu") (net 4))
+  (via (at 138.176 150.114) (size 0.7112) (drill 0.3048) (layers "F.Cu" "B.Cu") (net 4))
+  (segment (start 138.176 150.114) (end 138.176 118.11) (width 0.2032) (layer "B.Cu") (net 4))
+  (segment (start 138.176 118.11) (end 125.222 105.156) (width 0.2032) (layer "B.Cu") (net 4))
   (segment (start 125.931 147.772001) (end 125.931 150.008001) (width 0.2032) (layer "F.Cu") (net 6))
   (segment (start 125.981 145.486001) (end 125.981 147.722001) (width 0.2032) (layer "F.Cu") (net 6))

Commit message: Finish tracing
Parts:
- moved C3 1.56 mm to (137.8, 153.3)
- moved R7 1.56 mm to (137.8, 155.3)
Routing:
- net +3V3: track 190.3 -> 271.4 mm, vias 2 -> 5
- net Net-(SW6-Pad2): track 0.00 -> 80.6 mm, vias 0 -> 2
- net /CODEC_BITCLK: track 20.0 -> 76.4 mm, vias 0 -> 4
- net /CODEC_DATA_IN: track 17.3 -> 71.7 mm, vias 0 -> 2
- net /CODEC_DATA_OUT: track 16.3 -> 65.1 mm, vias 0 -> 4
- net /CODEC_A_OUT: track 0.00 -> 33.2 mm, vias 0 -> 3
- net /CODEC_A_IN: track 0.65 -> 15.5 mm, vias 0 -> 3
- net Net-(C5-Pad2): track 6.90 -> 10.6 mm
- net Net-(J1-Pad1): track 128.2 -> 131.8 mm
- net /RAW_IN: track 147.0 -> 148.9 mm
- net Net-(C3-Pad1): track 5.27 -> 4.67 mm
